File: DebugCAN_v3.brd (EAGLE design)
At the start: 56 x 80 mm, 47 parts, among them J1 RJHSE-5381-02, J3 MA04-1, J4 10118192-0001LF, U1 STM32F302C, U2 NCV7351D1E, U3 SI8621AB-B-IS, U4 AP2127N-3.3TRG1, U5 78L05F, U6 TLP291, U7 BH-9V-3P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

Commit message: final update
Parts:
- removed J4: 10118192-0001LF, con-usb:AMPHENOL_10118192-0001LF
- added D0: (no value), diode:SOD123
- added J2: 5077CR-16SMC2-BK-TR, 5077CR-16SMC2-BK-TR:NELTRON_5077CR-16SMC2-BK-TR
- added R1, R2: 5K1, rcl:R0603
- moved C6 7.07 mm to (46.7, 60.8), turned to 0 degrees
- moved TP4 5.31 mm to (41.2, 59.1)
- moved R5 4.95 mm to (44.1, 58.7)
- moved C12 4.21 mm to (37.4, 56.0), turned to 180 degrees
- moved U$1 3.95 mm to (19.0, 45.8), turned to 90 degrees
- moved U4 3.88 mm to (40.6, 54.7)
- moved TP1 3.76 mm to (46.5, 63.2)
- moved C7 3.75 mm to (36.6, 53.9)
- moved C13 3.70 mm to (25.7, 56.4), turned to 0 degrees
- moved TP5 3.56 mm to (42.2, 60.2)
- moved S1 3.38 mm to (29.4, 73.0), turned to 270 degrees
- moved U1 3.16 mm to (33.9, 59.5)
- moved TP2 3.13 mm to (37.6, 53.9)
- moved F1 3.00 mm to (21.4, 40.1)
- moved C10 2.86 mm to (40.6, 63.2)
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Connections:
- new net CC1: J2.A5, R1.2
- new net CC2: J2.B5, R2.1
- new net N$4: D0.A, U7.1
- net +5V: now also J2.A4_B9, J2.B4_A9; no longer J4.1
- net DCIN: now also D0.C; no longer U7.1
- net GNDA: now also J2.A1_B12, J2.B1_A12, J2.S1, J2.S2, J2.S3, J2.S4, R1.1, R2.2; no longer J4.4, J4.5, J4.SH1, J4.SH2, J4.SH3, J4.SH4, J4.SH5, J4.SH6
- net USB_DM: now also J2.A7, J2.B7; no longer J4.2
- net USB_DP: now also J2.A6, J2.B6; no longer J4.3
Routing:
- net N$4: track 0.00 -> 18.7 mm
- net DCIN: track 61.8 -> 43.6 mm
- net +5V: track 10.9 -> 19.3 mm, vias 1 -> 2
- net !RESET: track 22.6 -> 15.8 mm
- net CC1: track 0.00 -> 4.23 mm
- net EMS: track 38.5 -> 34.4 mm
- net CC2: track 0.00 -> 3.68 mm
- net CAN_LED: track 64.7 -> 61.2 mm
- net LED1: track 22.8 -> 19.9 mm
- net LED0: track 22.5 -> 19.7 mm
- net LED2: track 24.0 -> 21.2 mm
- net CANTX: track 18.9 -> 16.7 mm
- net USB_DM: track 11.8 -> 14.0 mm
- net SWCLK: track 7.72 -> 5.76 mm
- net N$11: track 8.59 -> 6.69 mm
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Other:
- board text added: "DebugCAN_ver3"
- board text added: "ver NHK2024-Ⅳ"
- board text removed: "DebugCAN"
- board text removed: "ver NHK2024-Ⅲ"
