File: DebugCAN_v3.sch (EAGLE design)
At the start: 47 parts, among them J1 RJHSE-5381-02, J3 MA04-1, J4 10118192-0001LF, U1 STM32F302C, U2 NCV7351D1E, U3 SI8621AB-B-IS, U4 AP2127N-3.3TRG1, U5 78L05F, U6 TLP291, U7 BH-9V-3P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

Commit message: final update
Parts:
- removed J4: 10118192-0001LF, con-usb:10118192-0001LF
- added D0: (no value), diode:DIODE-SOD123
- added J2: 5077CR-16SMC2-BK-TR, 5077CR-16SMC2-BK-TR:5077CR-16SMC2-BK-TR
- added R1, R2: 5K1, rcl:R-EU_R0603
Connections:
- new net CC1: J2.CC1, R1.2
- new net CC2: J2.CC2, R2.1
- new net N$4: D0.A, U7.1
- net +5V: now also J2.VBUS; no longer J4.VUSB
- net DCIN: now also D0.C; no longer U7.1
- net GNDA: now also J2.GND, J2.SHIELD, R1.1, R2.2; no longer J4.GND, J4.ID, J4.SHIELD
- net USB_DM: now also J2.DN1, J2.DN2; no longer J4.D-
- net USB_DP: now also J2.DP1, J2.DP2; no longer J4.D+
Changed lines of the file:
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@@
 <part name="GND52" library="supply1" library_urn="urn:adsk.eagle:library:371" deviceset="GNDIO" device=""/>
 <part name="U$1" library="con-xh" deviceset="XH-2-STRAIGHT" device=""/>
-<part name="GND32" library="supply1" library_urn="urn:adsk.eagle:library:371" deviceset="GNDA" device=""/>
-<part name="J4" library="con-usb" deviceset="10118192-0001LF" device=""/>
-<part name="P+14" library="supply1" library_urn="urn:adsk.eagle:library:371" deviceset="+5V" device=""/>
 <part name="GND7" library="supply1" library_urn="urn:adsk.eagle:library:371" deviceset="GNDIO" device=""/>
 <part name="P+3" library="supply1" library_urn="urn:adsk.eagle:library:371" deviceset="+12V" device=""/>
@@
 <part name="J1" library="con-rj45" deviceset="RJHSE-5381-02" device=""/>
 <part name="U7" library="BH-9V-3P" deviceset="BH-9V-3P" device=""/>
+<part name="D0" library="diode" library_urn="urn:adsk.eagle:library:210" deviceset="DIODE-" device="SOD123" package3d_urn="urn:adsk.eagle:package:43420/1"/>
+<part name="J2" library="5077CR-16SMC2-BK-TR" deviceset="5077CR-16SMC2-BK-TR" device=""/>
+<part name="GND4" library="supply1" library_urn="urn:adsk.eagle:library:371" deviceset="GNDA" device=""/>
+<part name="GND5" library="supply1" library_urn="urn:adsk.eagle:library:371" deviceset="GNDA" device=""/>
+<part name="P+6" library="supply1" library_urn="urn:adsk.eagle:library:371" deviceset="+5V" device=""/>
+<part name="R1" library="rcl" deviceset="R-EU_" device="R0603" value="5K1"/>
+<part name="GND6" library="supply1" library_urn="urn:adsk.eagle:library:371" deviceset="GNDA" device=""/>
+<part name="GND11" library="supply1" library_urn="urn:adsk.eagle:library:371" deviceset="GNDA" device=""/>
+<part name="R2" library="rcl" deviceset="R-EU_" device="R0603" value="5K1"/>
 </parts>
 <sheets>
@@
 <attribute name="NAME" x="224.79" y="109.22" size="1.778" layer="95" align="center-left"/>
 <attribute name="VALUE" x="224.79" y="106.68" size="1.778" layer="96" align="center-left"/>
+</instance>
+<instance part="D0" gate="G$1" x="200.66" y="101.6" smashed="yes" rot="R180">
+<attribute name="NAME" x="198.12" y="101.1174" size="1.778" layer="95" rot="R180"/>
+<attribute name="VALUE" x="198.12" y="103.9114" size="1.778" layer="96" rot="R180"/>
 </instance>
 </instances>
@@
 </net>
 <net name="DCIN" class="2">
-<segment>
-<wire x1="203.2" y1="101.6" x2="193.04" y2="101.6" width="0.1524" layer="91"/>
-<label x="193.04" y="101.6" size="1.778" layer="95" rot="R180"/>
-<pinref part="U7" gate="G$1" pin="1"/>
-</segment>
 <segment>
 <pinref part="F1" gate="G$1" pin="2"/>
@@
 <junction x="160.02" y="177.8"/>
 </segment>
+<segment>
+<pinref part="D0" gate="G$1" pin="C"/>
+<wire x1="198.12" y1="101.6" x2="187.96" y2="101.6" width="0.1524" layer="91"/>
+<label x="187.96" y="101.6" size="1.778" layer="95"/>
+</segment>
 </net>
 <net name="N$1" class="0">
@@
 <wire x1="210.82" y1="172.72" x2="205.74" y2="172.72" width="0.1524" layer="91"/>
 <pinref part="R11" gate="G$1" pin="2"/>
+</segment>
+</net>
+<net name="N$4" class="0">
+<segment>
+<pinref part="U7" gate="G$1" pin="1"/>
+<pinref part="D0" gate="G$1" pin="A"/>
 </segment>
 </net>
@@
 <attribute name="TP_SIGNAL_NAME" x="288.29" y="54.61" size="1.778" layer="97" rot="R90"/>
 </instance>
-<instance part="GND32" gate="1" x="238.76" y="7.62" smashed="yes">
-<attribute name="VALUE" x="236.22" y="5.08" size="1.778" layer="96" rot="R90"/>
-</instance>
-<instance part="J4" gate="G$1" x="215.9" y="5.08" smashed="yes" rot="R180">
-<attribute name="NAME" x="220.98618125" y="-5.601" size="1.780159375" layer="95" rot="R180"/>
-<attribute name="VALUE" x="220.988209375" y="17.8005" size="1.78086875" layer="96" rot="R180"/>
-</instance>
-<instance part="P+14" gate="1" x="246.38" y="-10.16" smashed="yes" rot="R270">
-<attribute name="VALUE" x="241.3" y="-7.62" size="1.778" layer="96"/>
+<instance part="J2" gate="G$1" x="302.26" y="0" smashed="yes">
+<attribute name="NAME" x="289.56" y="10.922" size="1.778" layer="95"/>
+<attribute name="VALUE" x="289.56" y="-15.24" size="1.778" layer="96"/>
+</instance>
+<instance part="GND4" gate="1" x="335.28" y="-10.16" smashed="yes" rot="R90">
+<attribute name="VALUE" x="337.82" y="-12.7" size="1.778" layer="96" rot="R180"/>
+</instance>
+<instance part="GND5" gate="1" x="269.24" y="-10.16" smashed="yes" rot="R270">
+<attribute name="VALUE" x="266.7" y="-7.62" size="1.778" layer="96"/>
+</instance>
+<instance part="P+6" gate="1" x="340.36" y="7.62" smashed="yes" rot="R270">
+<attribute name="VALUE" x="335.28" y="10.16" size="1.778" layer="96"/>
+</instance>
+<instance part="R1" gate="G$1" x="269.24" y="2.54" smashed="yes">
+<attribute name="NAME" x="265.43" y="4.0386" size="1.778" layer="95"/>
+<attribute name="VALUE" x="265.43" y="-0.762" size="1.778" layer="96"/>
+</instance>
+<instance part="GND6" gate="1" x="259.08" y="2.54" smashed="yes" rot="R270">
+<attribute name="VALUE" x="256.54" y="5.08" size="1.778" layer="96"/>
+</instance>
+<instance part="GND11" gate="1" x="347.98" y="-5.08" smashed="yes" rot="R90">
+<attribute name="VALUE" x="350.52" y="-7.62" size="1.778" layer="96" rot="R180"/>
+</instance>
+<instance part="R2" gate="G$1" x="337.82" y="-5.08" smashed="yes">
+<attribute name="NAME" x="334.01" y="-3.5814" size="1.778" layer="95"/>
+<attribute name="VALUE" x="334.01" y="-8.382" size="1.778" layer="96"/>
 </instance>
 </instances>
@@
 </segment>
 <segment>
-<label x="228.6" y="-2.54" size="1.778" layer="95"/>
-<wire x1="223.52" y1="0" x2="241.3" y2="0" width="0.1524" layer="91"/>
-<pinref part="J4" gate="G$1" pin="D-"/>
+<pinref part="J2" gate="G$1" pin="DN1"/>
+<wire x1="284.48" y1="-2.54" x2="274.32" y2="-2.54" width="0.1524" layer="91"/>
+<label x="274.32" y="-2.54" size="1.778" layer="95"/>
+</segment>
+<segment>
+<pinref part="J2" gate="G$1" pin="DN2"/>
+<wire x1="320.04" y1="0" x2="332.74" y2="0" width="0.1524" layer="91"/>
+<label x="322.58" y="0" size="1.778" layer="95"/>
 </segment>
 </net>
@@
 </segment>
 <segment>
-<wire x1="246.38" y1="2.54" x2="223.52" y2="2.54" width="0.1524" layer="91"/>
-<pinref part="J4" gate="G$1" pin="D+"/>
-<label x="233.68" y="5.08" size="1.778" layer="95" rot="R180"/>
+<pinref part="J2" gate="G$1" pin="DP1"/>
+<wire x1="284.48" y1="0" x2="274.32" y2="0" width="0.1524" layer="91"/>
+<label x="274.32" y="0" size="1.778" layer="95"/>
+</segment>
+<segment>
+<pinref part="J2" gate="G$1" pin="DP2"/>
+<wire x1="320.04" y1="-2.54" x2="332.74" y2="-2.54" width="0.1524" layer="91"/>
+<label x="322.58" y="-2.54" size="1.778" layer="95"/>
 </segment>
 </net>
@@
 </segment>
 <segment>
-<pinref part="GND32" gate="1" pin="GNDA"/>
-<wire x1="226.06" y1="12.7" x2="238.76" y2="12.7" width="0.1524" layer="91"/>
-<wire x1="238.76" y1="12.7" x2="238.76" y2="10.16" width="0.1524" layer="91"/>
-<wire x1="223.52" y1="7.62" x2="226.06" y2="7.62" width="0.1524" layer="91"/>
-<wire x1="226.06" y1="7.62" x2="226.06" y2="12.7" width="0.1524" layer="91"/>
-<pinref part="J4" gate="G$1" pin="GND"/>
-<pinref part="J4" gate="G$1" pin="SHIELD"/>
-<wire x1="223.52" y1="12.7" x2="226.06" y2="12.7" width="0.1524" layer="91"/>
-<junction x="226.06" y="12.7"/>
-<pinref part="J4" gate="G$1" pin="ID"/>
-<wire x1="223.52" y1="5.08" x2="226.06" y2="5.08" width="0.1524" layer="91"/>
-<wire x1="226.06" y1="5.08" x2="226.06" y2="7.62" width="0.1524" layer="91"/>
-<junction x="226.06" y="7.62"/>
+<pinref part="GND4" gate="1" pin="GNDA"/>
+<wire x1="320.04" y1="-10.16" x2="332.74" y2="-10.16" width="0.1524" layer="91"/>
+<pinref part="J2" gate="G$1" pin="GND"/>
+</segment>
+<segment>
+<pinref part="GND5" gate="1" pin="GNDA"/>
+<wire x1="284.48" y1="-10.16" x2="271.78" y2="-10.16" width="0.1524" layer="91"/>
+<pinref part="J2" gate="G$1" pin="SHIELD"/>
+</segment>
+<segment>
+<wire x1="264.16" y1="2.54" x2="261.62" y2="2.54" width="0.1524" layer="91"/>
+<pinref part="GND6" gate="1" pin="GNDA"/>
+<pinref part="R1" gate="G$1" pin="1"/>
+</segment>
+<segment>
+<pinref part="GND11" gate="1" pin="GNDA"/>
+<pinref part="R2" gate="G$1" pin="2"/>
+<wire x1="345.44" y1="-5.08" x2="342.9" y2="-5.08" width="0.1524" layer="91"/>
 </segment>
 </net>
@@
 </segment>
 <segment>
-<pinref part="J4" gate="G$1" pin="VUSB"/>
-<wire x1="223.52" y1="-2.54" x2="226.06" y2="-2.54" width="0.1524" layer="91"/>
-<wire x1="226.06" y1="-2.54" x2="226.06" y2="-10.16" width="0.1524" layer="91"/>
-<wire x1="226.06" y1="-10.16" x2="243.84" y2="-10.16" width="0.1524" layer="91"/>
-<pinref part="P+14" gate="1" pin="+5V"/>
+<wire x1="320.04" y1="7.62" x2="337.82" y2="7.62" width="0.1524" layer="91"/>
+<pinref part="P+6" gate="1" pin="+5V"/>
+<pinref part="J2" gate="G$1" pin="VBUS"/>
 </segment>
 </net>
@@
 </segment>
 </net>
+<net name="CC2" class="0">
+<segment>
+<pinref part="J2" gate="G$1" pin="CC2"/>
+<wire x1="320.04" y1="-5.08" x2="332.74" y2="-5.08" width="0.1524" layer="91"/>
+<label x="327.66" y="-5.08" size="1.778" layer="95"/>
+<pinref part="R2" gate="G$1" pin="1"/>
+</segment>
+</net>
+<net name="CC1" class="0">
+<segment>
+<pinref part="J2" gate="G$1" pin="CC1"/>
+<wire x1="284.48" y1="2.54" x2="274.32" y2="2.54" width="0.1524" layer="91"/>
+<pinref part="R1" gate="G$1" pin="2"/>
+<label x="279.4" y="2.54" size="1.778" layer="95"/>
+</segment>
+</net>
